Commit message: Add files via upload

File: src/gofr_description/urdf/gofr.urdf.xacro (robot description, xacro)
@@ -13,5 +13,5 @@
       <origin rpy="0 0 0" xyz="0 0 0"/>
       <geometry>
-        <mesh filename="package://gofr_description/meshes/bases/base_link_m-binary.stl"/>
+        <mesh filename="package://gofr_description/meshes/bases/GOFR_mini.stl"/>
       </geometry>
       <material name="light_black"/>
@@ -20,10 +20,10 @@
       <origin xyz="0 0 0" rpy="0 0 0"/>
       <geometry>
-        <mesh filename="package://gofr_description/meshes/bases/base_link_m-binary.stl"/>
+        <mesh filename="package://gofr_description/meshes/bases/GOFR_mini.stl"/>
       </geometry>
     </collision>
     <inertial>
       <origin rpy="0 0 0" xyz="5.834560042719257e-07 7.554645109307412e-16 0.13547716753400393"/>
-      <mass value="442.4085411014063"/>
+      <mass value="4.5"/>
       <inertia ixx="10.851545" ixy="0.0" ixz="-8.3e-05"
                iyy="20.978869" iyz="-0.0"
@@ -31,5 +31,5 @@
     </inertial>
   </link>
-  <joint name="wheel_front_left_joint" type="fixed">
+  <!-- <joint name="wheel_front_left_joint" type="fixed">
     <parent link="base_link"/>
     <child link="wheel_front_left_link"/>
@@ -211,5 +211,5 @@
       <inertia ixx="1.137646" ixy="0.0" ixz="0.123419" iyy="1.044686" iyz="0.0" izz="0.262287"/>
     </inertial>
-  </link>
+  </link> -->
   <joint name="imu_joint" type="fixed">
     <parent link="base_link"/>

Commit message: Moved Camera and Updated Gazebo world

File: src/gofr_description/urdf/gofr.urdf.xacro (robot description, xacro)
@@ -135,5 +135,5 @@
     </inertial>
   </link>
-  <joint name="forks_joint" type="fixed">
+  <joint name="forks_joint" type="prismatic">
     <parent link="forks_base_link"/>
     <child link="forks_link"/>
@@ -245,11 +245,11 @@
   </link>
   <joint name="camera_joint" type="fixed">
-    <origin xyz="0.073 -0.011 0.084" rpy="0 0 0"/>
-    <parent link="base_link"/>
+    <origin xyz="0 -0.108217 .03" rpy="0 0 0"/>
+    <parent link="lift_link"/>
     <child link="camera_link"/>
   </joint>
   <link name="camera_link">
     <collision>
-      <origin xyz="0.005 0.011 0.013" rpy="0 0 0"/>
+      <origin xyz="0 0 0" rpy="0 0 0"/>
       <geometry>
         <box size="0.015 0.030 0.027"/>
