Commit message: Simulation Actuators

File: src/gofr_description/urdf/gofr.gazebo.xacro (robot description, xacro)
@@ -74,5 +74,5 @@
     <minDepth>0.001</minDepth>
     <maxVel>0.1</maxVel>
-    <fdir1>1 0 0</fdir1>
+    <fdir1>0 0 1</fdir1>
     <material>Gazebo/FlatBlack</material>
   </gazebo>

File: src/gofr_description/urdf/gofr.urdf.xacro (robot description, xacro)
@@ -135,5 +135,5 @@
     </inertial>
   </link>
-  <joint name="forks_joint" type="prismatic">
+  <joint name="forks_joint" type="fixed">
     <parent link="forks_base_link"/>
     <child link="forks_link"/>
@@ -186,10 +186,21 @@
     </inertial>
   </link>
-  <joint name="lift_joint" type="fixed">
+  <joint name="lift_joint" type="prismatic">
     <parent link="base_link"/>
     <child link="lift_link"/>
     <origin xyz="1.3e-05 0.108217 0.758685" rpy="0 0 0"/>
     <axis xyz="0 0 0.01"/>
-  </joint>
+    <limit effort="100" lower="0.0" upper="0.4572" velocity="100"/>
+  </joint>
+<transmission name="lift_tran">
+    <type>transmission_interface/SimpleTransmission</type>
+    <joint name="lift_joint">
+      <hardwareInterface>hardware_interface/PositionJointInterface</hardwareInterface>
+    </joint>
+    <actuator name="lift_actr">
+      <hardwareInterface>hardware_interface/PositionJointInterface</hardwareInterface>
+      <mechanicalReduction>1</mechanicalReduction>
+    </actuator>
+  </transmission>
   <link name="lift_link">
     <visual>
